Commit message: Add files via upload

File: src/bumperbot_description/urdf/bumperbot.urdf.xacro (robot description, xacro)
@@ -1,6 +1,14 @@
 <?xml version="1.0"?>
-<robot xmlns:xacro="http://www.ros.org/wiki.xacro" name="bumperbot">
+<robot xmlns:xacro="http://www.ros.org/wiki/xacro" name="bumperbot">
+    <xacro:include filename="$(find bumperbot_description)/urdf/bumperbot_gazebo.xacro" />
     <link name="base_footprint"/>
     <link name="base_link">
+        <inertial>
+            <origin xyz="0 0 0.04" rpy="0.0 0.25 0.3" />
+            <mass value="8.2573504e-01"/>
+            <inertia ixx="2.2124416e-02" ixy="-1.2294101e-04" ixz="3.4938785e-04"
+                    iyy="2.1193702e-02" iyz="-5.0120904e-05"
+                    izz="2.0064271e-02" />
+        </inertial>
         <visual>
             <origin rpy="0 0 0" xyz="0 0 0"/>
@@ -9,4 +17,10 @@
             </geometry>
         </visual>
+        <collision>
+            <origin rpy="0 0 0" xyz="0 0 0"/>
+            <geometry>
+                <mesh filename="package://bumperbot_description/meshes/base_link.STL"/>
+            </geometry>
+        </collision>
     </link>
     <joint name="base_joint" type="fixed">
@@ -16,4 +30,11 @@
     </joint>
     <link name="wheel_right_link">
+        <inertial>
+            <origin xyz="0 0 0.04" rpy="0.0 0.25 0.3" />
+            <mass value="8.2573504e-01"/>
+            <inertia ixx="2.2124416e-02" ixy="-1.2294101e-04" ixz="3.4938785e-04"
+                    iyy="2.1193702e-02" iyz="-5.0120904e-05"
+                    izz="2.0064271e-02" />
+        </inertial>
         <visual>
             <origin rpy="1.57 0 0" xyz="0 0 0"/>
@@ -22,4 +43,10 @@
             </geometry>
         </visual>
+        <collision>
+            <origin xyz="0 -0.015 0" rpy="1.57 0 0"/>
+            <geometry>
+                <sphere radius="0.033"/>
+            </geometry>
+        </collision>
     </link>
     <joint name="wheel_right_joint" type="continuous">
@@ -30,4 +57,11 @@
     </joint>
     <link name="wheel_left_link">
+        <inertial>
+            <origin xyz="0 0 0.04" rpy="0.0 0.25 0.3" />
+            <mass value="8.2573504e-01"/>
+            <inertia ixx="2.2124416e-02" ixy="-1.2294101e-04" ixz="3.4938785e-04"
+                    iyy="2.1193702e-02" iyz="-5.0120904e-05"
+                    izz="2.0064271e-02" />
+        </inertial>
         <visual>
             <origin rpy="-1.57 0 0" xyz="0 0 0"/>
@@ -36,4 +70,10 @@
             </geometry>
         </visual>
+        <collision>
+            <origin xyz="0 0.015 0" rpy="1.57 0 0"/>
+            <geometry>
+                <sphere radius="0.033"/>
+            </geometry>
+        </collision>
     </link>
     <joint name="wheel_left_joint" type="continuous">
@@ -44,4 +84,11 @@
     </joint>
     <link name="caster_front_link">
+        <inertial>
+            <origin xyz="0 0 0.04" rpy="0.0 0.25 0.3" />
+            <mass value="8.2573504e-01"/>
+            <inertia ixx="2.2124416e-02" ixy="-1.2294101e-04" ixz="3.4938785e-04"
+                    iyy="2.1193702e-02" iyz="-5.0120904e-05"
+                    izz="2.0064271e-02" />
+        </inertial>
         <visual>
             <origin rpy="0 0 0" xyz="0 0 0"/>
@@ -50,4 +97,10 @@
             </geometry>
         </visual>
+        <collision>
+            <origin xyz="0 0 0" rpy="0 0 0"/>
+            <geometry>
+                <sphere radius="0.005"/>
+            </geometry>
+        </collision>
     </link>
     <joint name="caster_front_joint" type="fixed">
@@ -57,4 +110,11 @@
     </joint>
     <link name="caster_rear_link">
+        <inertial>
+            <origin xyz="0 0 0.04" rpy="0.0 0.25 0.3" />
+            <mass value="8.2573504e-01"/>
+            <inertia ixx="2.2124416e-02" ixy="-1.2294101e-04" ixz="3.4938785e-04"
+                    iyy="2.1193702e-02" iyz="-5.0120904e-05"
+                    izz="2.0064271e-02" />
+        </inertial>
         <visual>
             <origin rpy="0 0 0" xyz="0 0 0"/>
@@ -63,4 +123,10 @@
             </geometry>
         </visual>
+        <collision>
+            <origin xyz="0 0 0" rpy="0 0 0"/>
+            <geometry>
+                <sphere radius="0.005"/>
+            </geometry>
+        </collision>
     </link>
     <joint name="caster_rear_joint" type="fixed">
